File: electronics/_saved_microbit-extension.sch (KiCad schematic (older format))
At the start: 26 parts, among them SW1 SW_DIP_x01, SW2 SW_DIP_x01, SW3 SW_DIP_x01, SW4 SW_DIP_x01

Commit message: exported pdf
Parts:
- removed Q?: 2N7002, TO_SOT_Packages_SMD:SOT-23, symbol 2N7002
- added D?: D, symbol D
- added R? (x2): 1K, symbol R
- added T?: 2N4401, TO92-CBE, symbol 2N4401
- added U?: LM1084IS-3.3/NOPB, TO_SOT_Packages_SMD:TO-263-3Lead, symbol LM1084IS-3.3/NOPB
Connections:
- net labels added: BUZZER_PIN
- wire segments 48 -> 55
Other:
- moved on the sheet: BZ?
Changed lines of the file:
@@
 LIBS:switches
 LIBS:TLC5917ID
+LIBS:2N4401
 LIBS:microbit-extension-cache
 EELAYER 25 0
@@
 L Buzzer BZ?
 U 1 1 598737DA
-P 10500 5300
-F 0 "BZ?" H 10650 5350 50  0000 L CNN
-F 1 "Buzzer" H 10650 5250 50  0000 L CNN
-F 2 "" V 10475 5400 50  0001 C CNN
-F 3 "" V 10475 5400 50  0001 C CNN
-	1    10500 5300
-	1    0    0    -1
-$EndComp
-$Comp
-L 2N7002 Q?
-U 1 1 59873A0C
-P 10300 5750
-F 0 "Q?" H 10500 5825 50  0000 L CNN
-F 1 "2N7002" H 10500 5750 50  0000 L CNN
-F 2 "TO_SOT_Packages_SMD:SOT-23" H 10500 5675 50  0001 L CIN
-F 3 "" H 10300 5750 50  0001 L CNN
-	1    10300 5750
-	1    0    0    -1
-$EndComp
+P 10750 5450
+F 0 "BZ?" H 10900 5500 50  0000 L CNN
+F 1 "Buzzer" H 10900 5400 50  0000 L CNN
+F 2 "" V 10725 5550 50  0001 C CNN
+F 3 "" V 10725 5550 50  0001 C CNN
+	1    10750 5450
+	1    0    0    -1
+$EndComp
+$Comp
+L 2N4401 T?
+U 1 1 59873D13
+P 10350 5850
+F 0 "T?" H 9949 6150 50  0000 L BNN
+F 1 "2N4401" H 9950 6050 50  0000 L BNN
+F 2 "TO92-CBE" H 10350 5850 50  0001 L BNN
+F 3 "Multicomp" H 10350 5850 50  0001 L BNN
+F 4 "BIPOLAR TRANSISTOR%2C NPN%2C TO-92%3B Transistor Polarity%3A NPN%3B Collector Emitter Voltage V%28br%29ceo%3A 40V%3B Transition Frequen..." H 10350 5850 50  0001 L BNN "Description"
+F 5 "0.14 USD" H 10350 5850 50  0001 L BNN "Price"
+F 6 "2N4401" H 10350 5850 50  0001 L BNN "MP"
+F 7 "Good" H 10350 5850 50  0001 L BNN "Availability"
+F 8 "TO-92 Multicomp" H 10350 5850 50  0001 L BNN "Package"
+	1    10350 5850
+	1    0    0    -1
+$EndComp
+Wire Wire Line
+	10450 5500 10450 5650
+Wire Wire Line
+	10450 5550 10650 5550
+$Comp
+L D D?
+U 1 1 59873EE7
+P 10450 5350
+F 0 "D?" H 10450 5450 50  0000 C CNN
+F 1 "D" H 10450 5250 50  0000 C CNN
+F 2 "" H 10450 5350 50  0001 C CNN
+F 3 "" H 10450 5350 50  0001 C CNN
+	1    10450 5350
+	0    1    1    0
+$EndComp
+Connection ~ 10450 5550
+$Comp
+L R R?
+U 1 1 59873FD2
+P 10450 5000
+F 0 "R?" V 10530 5000 50  0000 C CNN
+F 1 "1K" V 10450 5000 50  0000 C CNN
+F 2 "" V 10380 5000 50  0001 C CNN
+F 3 "" H 10450 5000 50  0001 C CNN
+	1    10450 5000
+	1    0    0    -1
+$EndComp
+Wire Wire Line
+	10450 5150 10450 5200
+Wire Wire Line
+	10650 4850 10650 5350
+Wire Wire Line
+	10000 4850 10650 4850
+Connection ~ 10450 4850
+$Comp
+L +3.3V #PWR?
+U 1 1 598742F8
+P 10000 4850
+F 0 "#PWR?" H 10000 4700 50  0001 C CNN
+F 1 "+3.3V" H 10000 4990 50  0000 C CNN
+F 2 "" H 10000 4850 50  0001 C CNN
+F 3 "" H 10000 4850 50  0001 C CNN
+	1    10000 4850
+	0    -1   -1   0
+$EndComp
+$Comp
+L R R?
+U 1 1 59874535
+P 10050 5850
+F 0 "R?" V 10130 5850 50  0000 C CNN
+F 1 "1K" V 10050 5850 50  0000 C CNN
+F 2 "" V 9980 5850 50  0001 C CNN
+F 3 "" H 10050 5850 50  0001 C CNN
+	1    10050 5850
+	0    1    1    0
+$EndComp
+Wire Wire Line
+	10200 5850 10250 5850
+$Comp
+L GND #PWR?
+U 1 1 5987477E
+P 10450 6050
+F 0 "#PWR?" H 10450 5800 50  0001 C CNN
+F 1 "GND" H 10450 5900 50  0000 C CNN
+F 2 "" H 10450 6050 50  0001 C CNN
+F 3 "" H 10450 6050 50  0001 C CNN
+	1    10450 6050
+	1    0    0    -1
+$EndComp
+Wire Wire Line
+	9350 5850 9900 5850
+Text Label 9350 5850 0    60   ~ 0
+BUZZER_PIN
+$Comp
+L LM1084IS-3.3/NOPB U?
+U 1 1 59874ABB
+P 5250 5600
+F 0 "U?" H 5450 5400 50  0000 C CNN
+F 1 "LM1084IS-3.3/NOPB" H 4950 5800 50  0000 L CNN
+F 2 "TO_SOT_Packages_SMD:TO-263-3Lead" H 5250 5700 50  0001 C CIN
+F 3 "" H 5250 5600 50  0001 C CNN
+	1    5250 5600
+	1    0    0    -1
+$EndComp

Commit message: more updates to schematics
Parts:
- removed U?: LM1084IS-3.3/NOPB, TO_SOT_Packages_SMD:TO-263-3Lead, symbol LM1084IS-3.3/NOPB
- added C? (x2): C, symbol C
- added U?: LD1117S33CTR, TO_SOT_Packages_SMD:SOT-223, symbol LD1117S33CTR
Connections:
- net labels added: +9V
- wire segments 55 -> 61
Changed lines of the file:
@@
 BUZZER_PIN
 $Comp
-L LM1084IS-3.3/NOPB U?
-U 1 1 59874ABB
-P 5250 5600
-F 0 "U?" H 5450 5400 50  0000 C CNN
-F 1 "LM1084IS-3.3/NOPB" H 4950 5800 50  0000 L CNN
-F 2 "TO_SOT_Packages_SMD:TO-263-3Lead" H 5250 5700 50  0001 C CIN
-F 3 "" H 5250 5600 50  0001 C CNN
-	1    5250 5600
+L LD1117S33CTR U?
+U 1 1 59874CBE
+P 8700 4150
+F 0 "U?" H 8700 4400 50  0000 C CNN
+F 1 "LD1117S33CTR" H 8700 4350 50  0000 C CNN
+F 2 "TO_SOT_Packages_SMD:SOT-223" H 8700 4250 50  0001 C CNN
+F 3 "" H 8700 4150 50  0001 C CNN
+	1    8700 4150
 	1    0    0    -1
 $EndComp
+Wire Wire Line
+	8700 4400 8700 4700
+$Comp
+L GND #PWR?
+U 1 1 598750F5
+P 8700 4700
+F 0 "#PWR?" H 8700 4450 50  0001 C CNN
+F 1 "GND" H 8700 4550 50  0000 C CNN
+F 2 "" H 8700 4700 50  0001 C CNN
+F 3 "" H 8700 4700 50  0001 C CNN
+	1    8700 4700
+	1    0    0    -1
+$EndComp
+Wire Wire Line
+	7900 4100 8300 4100
+$Comp
+L C C?
+U 1 1 59875242
+P 8150 4400
+F 0 "C?" H 8175 4500 50  0000 L CNN
+F 1 "C" H 8175 4300 50  0000 L CNN
+F 2 "" H 8188 4250 50  0001 C CNN
+F 3 "" H 8150 4400 50  0001 C CNN
+	1    8150 4400
+	1    0    0    -1
+$EndComp
+$Comp
+L C C?
+U 1 1 598752C6
+P 9200 4400
+F 0 "C?" H 9225 4500 50  0000 L CNN
+F 1 "C" H 9225 4300 50  0000 L CNN
+F 2 "" H 9238 4250 50  0001 C CNN
+F 3 "" H 9200 4400 50  0001 C CNN
+	1    9200 4400
+	1    0    0    -1
+$EndComp
+Wire Wire Line
+	9100 4100 9550 4100
+Wire Wire Line
+	8150 4100 8150 4250
+Connection ~ 8150 4100
+Wire Wire Line
+	9200 4100 9200 4250
+Connection ~ 9200 4100
+Wire Wire Line
+	8150 4550 9200 4550
+Connection ~ 8700 4550
+$Comp
+L +9V #PWR?
+U 1 1 59875598
+P 7900 4100
+F 0 "#PWR?" H 7900 3950 50  0001 C CNN
+F 1 "+9V" H 7900 4240 50  0000 C CNN
+F 2 "" H 7900 4100 50  0001 C CNN
+F 3 "" H 7900 4100 50  0001 C CNN
+	1    7900 4100
+	0    -1   -1   0
+$EndComp
+$Comp
+L +3.3V #PWR?
+U 1 1 598756CA
+P 9550 4100
+F 0 "#PWR?" H 9550 3950 50  0001 C CNN
+F 1 "+3.3V" H 9550 4240 50  0000 C CNN
+F 2 "" H 9550 4100 50  0001 C CNN
+F 3 "" H 9550 4100 50  0001 C CNN
+	1    9550 4100
+	0    1    1    0
+$EndComp
 $EndSCHEMATC
