File: electronics/microbit-extension.sch (KiCad schematic (older format))
At the start: 31 parts, among them J1 microbit_edge_connector, J2 9V conn, SW1 SW_DIP_x01, SW2 SW_DIP_x01, SW3 SW_DIP_x01, SW4 SW_DIP_x01, T1 2N4401, U1 LD1117S33CTR

Commit message: updated to schematics
Parts:
- BZ1: footprint Buzzers_Beepers:BUZZER -> footprints:BUZZER
- C1, C2: footprint Capacitors_SMD:C_0805 -> footprints:C_0805
- D1, D2, D3, D4, D5: footprint LEDs:LED_D3.0mm -> footprints:LED_D3.0mm
- D6: footprint LEDs:LED_RGB_5050-6 -> footprints:LED_RGB_5050-6
- J1: footprint Connectors_4UCON:4UCON_17909_02x401.27mm_Vertical -> footprints:4UCON_17909_02x401.27mm_Vertical
- J2: footprint Pin_Headers:Pin_Header_Straight_1x02_Pitch2.54mm -> footprints:Pin_Header_Straight_1x02_Pitch2.54mm
- R1, R10, R11, R12, R13, R2, R3, R4, R5, R6, R7, R8, R9: footprint Resistors_SMD:R_0805 -> footprints:R_0805
- RV1: footprint Potentiometers:Potentiometer_Alps_RK09K_Horizontal -> footprints:Potentiometer_Alps_RK09K_Horizontal
- SW1, SW2, SW3, SW4: footprint Buttons_Switches_SMD:SW_SPST_EVPBF -> footprints:SW_SPST_EVPBF
- T1: footprint TO_SOT_Packages_SMD:SOT-23 -> footprints:SOT-23; symbol 2N4401 -> 2N4401-RESCUE-microbit-extension
- U1: footprint TO_SOT_Packages_SMD:SOT-223 -> footprints:SOT-223
Connections:
- net GND: now also T1.2; no longer T1.E
- net at BZ1.2 (+): now also T1.3; no longer T1.C
- net at R9.1: now also T1.1; no longer T1.B
Changed lines of the file:
@@
 EESchema Schematic File Version 2
+LIBS:microbit-extension-rescue
 LIBS:power
 LIBS:device
@@
 F 0 "J1" H 1350 4700 50  0000 C CNN
 F 1 "microbit_edge_connector" H 1350 4600 50  0000 C CNN
-F 2 "Connectors_4UCON:4UCON_17909_02x401.27mm_Vertical" H 1200 2550 50  0001 C CNN
+F 2 "footprints:4UCON_17909_02x401.27mm_Vertical" H 1200 2550 50  0001 C CNN
 F 3 "" H 1200 2550 50  0001 C CNN
 	1    1300 2650
@@
 F 0 "SW1" H 10600 1600 50  0000 C CNN
 F 1 "SW_DIP_x01" H 10600 1300 50  0000 C CNN
-F 2 "Buttons_Switches_SMD:SW_SPST_EVPBF" H 10600 1450 50  0001 C CNN
+F 2 "footprints:SW_SPST_EVPBF" H 10600 1450 50  0001 C CNN
 F 3 "" H 10600 1450 50  0001 C CNN
 	1    10600 1450
@@
 F 0 "R10" V 10230 1250 50  0000 C CNN
 F 1 "R" V 10150 1250 50  0000 C CNN
-F 2 "Resistors_SMD:R_0805" V 10080 1250 50  0001 C CNN
+F 2 "footprints:R_0805" V 10080 1250 50  0001 C CNN
 F 3 "" H 10150 1250 50  0001 C CNN
 	1    10150 1250
@@
 F 0 "SW2" H 10600 2150 50  0000 C CNN
 F 1 "SW_DIP_x01" H 10600 1850 50  0000 C CNN
-F 2 "Buttons_Switches_SMD:SW_SPST_EVPBF" H 10600 2000 50  0001 C CNN
+F 2 "footprints:SW_SPST_EVPBF" H 10600 2000 50  0001 C CNN
 F 3 "" H 10600 2000 50  0001 C CNN
 	1    10600 2000
@@
 F 0 "R11" V 10230 1800 50  0000 C CNN
 F 1 "R" V 10150 1800 50  0000 C CNN
-F 2 "Resistors_SMD:R_0805" V 10080 1800 50  0001 C CNN
+F 2 "footprints:R_0805" V 10080 1800 50  0001 C CNN
 F 3 "" H 10150 1800 50  0001 C CNN
 	1    10150 1800
@@
 F 0 "SW3" H 10600 2700 50  0000 C CNN
 F 1 "SW_DIP_x01" H 10600 2400 50  0000 C CNN
-F 2 "Buttons_Switches_SMD:SW_SPST_EVPBF" H 10600 2550 50  0001 C CNN
+F 2 "footprints:SW_SPST_EVPBF" H 10600 2550 50  0001 C CNN
 F 3 "" H 10600 2550 50  0001 C CNN
 	1    10600 2550
@@
 F 0 "R12" V 10230 2350 50  0000 C CNN
 F 1 "R" V 10150 2350 50  0000 C CNN
-F 2 "Resistors_SMD:R_0805" V 10080 2350 50  0001 C CNN
+F 2 "footprints:R_0805" V 10080 2350 50  0001 C CNN
 F 3 "" H 10150 2350 50  0001 C CNN
 	1    10150 2350
@@
 F 0 "SW4" H 10600 3150 50  0000 C CNN
 F 1 "SW_DIP_x01" H 10600 2850 50  0000 C CNN
-F 2 "Buttons_Switches_SMD:SW_SPST_EVPBF" H 10600 3000 50  0001 C CNN
+F 2 "footprints:SW_SPST_EVPBF" H 10600 3000 50  0001 C CNN
 F 3 "" H 10600 3000 50  0001 C CNN
 	1    10600 3000
@@
 F 0 "R13" V 10230 2800 50  0000 C CNN
 F 1 "R" V 10150 2800 50  0000 C CNN
-F 2 "Resistors_SMD:R_0805" V 10080 2800 50  0001 C CNN
+F 2 "footprints:R_0805" V 10080 2800 50  0001 C CNN
 F 3 "" H 10150 2800 50  0001 C CNN
 	1    10150 2800
@@
 F 0 "RV1" V 10425 4150 50  0000 C CNN
 F 1 "POT" V 10500 4150 50  0000 C CNN
-F 2 "Potentiometers:Potentiometer_Alps_RK09K_Horizontal" H 10600 4150 50  0001 C CNN
+F 2 "footprints:Potentiometer_Alps_RK09K_Horizontal" H 10600 4150 50  0001 C CNN
 F 3 "" H 10600 4150 50  0001 C CNN
 	1    10600 4150
@@
 F 0 "D1" H 8800 1250 50  0000 C CNN
 F 1 "LED" H 8800 1050 50  0000 C CNN
-F 2 "LEDs:LED_D3.0mm" H 8800 1150 50  0001 C CNN
+F 2 "footprints:LED_D3.0mm" H 8800 1150 50  0001 C CNN
 F 3 "" H 8800 1150 50  0001 C CNN
 	1    8800 1150
@@
 F 0 "R1" V 8430 1150 50  0000 C CNN
 F 1 "R" V 8350 1150 50  0000 C CNN
-F 2 "Resistors_SMD:R_0805" V 8280 1150 50  0001 C CNN
+F 2 "footprints:R_0805" V 8280 1150 50  0001 C CNN
 F 3 "" H 8350 1150 50  0001 C CNN
 	1    8350 1150
@@
 F 0 "D3" H 8800 1850 50  0000 C CNN
 F 1 "LED" H 8800 1650 50  0000 C CNN
-F 2 "LEDs:LED_D3.0mm" H 8800 1750 50  0001 C CNN
+F 2 "footprints:LED_D3.0mm" H 8800 1750 50  0001 C CNN
 F 3 "" H 8800 1750 50  0001 C CNN
 	1    8800 1750
@@
 F 0 "R3" V 8430 1750 50  0000 C CNN
 F 1 "R" V 8350 1750 50  0000 C CNN
-F 2 "Resistors_SMD:R_0805" V 8280 1750 50  0001 C CNN
+F 2 "footprints:R_0805" V 8280 1750 50  0001 C CNN
 F 3 "" H 8350 1750 50  0001 C CNN
 	1    8350 1750
@@
 F 0 "D2" H 8800 1550 50  0000 C CNN
 F 1 "LED" H 8800 1350 50  0000 C CNN
-F 2 "LEDs:LED_D3.0mm" H 8800 1450 50  0001 C CNN
+F 2 "footprints:LED_D3.0mm" H 8800 1450 50  0001 C CNN
 F 3 "" H 8800 1450 50  0001 C CNN
 	1    8800 1450
@@
 F 0 "R2" V 8430 1450 50  0000 C CNN
 F 1 "R" V 8350 1450 50  0000 C CNN
-F 2 "Resistors_SMD:R_0805" V 8280 1450 50  0001 C CNN
+F 2 "footprints:R_0805" V 8280 1450 50  0001 C CNN
 F 3 "" H 8350 1450 50  0001 C CNN
 	1    8350 1450
@@
 F 0 "D4" H 8800 2150 50  0000 C CNN
 F 1 "LED" H 8800 1950 50  0000 C CNN
-F 2 "LEDs:LED_D3.0mm" H 8800 2050 50  0001 C CNN
+F 2 "footprints:LED_D3.0mm" H 8800 2050 50  0001 C CNN
 F 3 "" H 8800 2050 50  0001 C CNN
 	1    8800 2050
@@
 F 0 "R4" V 8430 2050 50  0000 C CNN
 F 1 "R" V 8350 2050 50  0000 C CNN
-F 2 "Resistors_SMD:R_0805" V 8280 2050 50  0001 C CNN
+F 2 "footprints:R_0805" V 8280 2050 50  0001 C CNN
 F 3 "" H 8350 2050 50  0001 C CNN
 	1    8350 2050
@@
 F 0 "D5" H 8800 2450 50  0000 C CNN
 F 1 "LED" H 8800 2250 50  0000 C CNN
-F 2 "LEDs:LED_D3.0mm" H 8800 2350 50  0001 C CNN
+F 2 "footprints:LED_D3.0mm" H 8800 2350 50  0001 C CNN
 F 3 "" H 8800 2350 50  0001 C CNN
 	1    8800 2350
@@
 F 0 "R5" V 8430 2350 50  0000 C CNN
 F 1 "R" V 8350 2350 50  0000 C CNN
-F 2 "Resistors_SMD:R_0805" V 8280 2350 50  0001 C CNN
+F 2 "footprints:R_0805" V 8280 2350 50  0001 C CNN
 F 3 "" H 8350 2350 50  0001 C CNN
 	1    8350 2350
@@
 F 0 "D6" H 8800 3320 50  0000 C CNN
 F 1 "LED_RGB" H 8800 2600 50  0000 C CNN
-F 2 "LEDs:LED_RGB_5050-6" H 8800 2900 50  0001 C CNN
+F 2 "footprints:LED_RGB_5050-6" H 8800 2900 50  0001 C CNN
 F 3 "" H 8800 2900 50  0001 C CNN
 	1    8800 2950
@@
 F 0 "R6" V 8250 2750 50  0000 C CNN
 F 1 "R" V 8350 2750 50  0000 C CNN
-F 2 "Resistors_SMD:R_0805" V 8280 2750 50  0001 C CNN
+F 2 "footprints:R_0805" V 8280 2750 50  0001 C CNN
 F 3 "" H 8350 2750 50  0001 C CNN
 	1    8350 2750
@@
 F 0 "R7" V 8250 2950 50  0000 C CNN
 F 1 "R" V 8350 2950 50  0000 C CNN
-F 2 "Resistors_SMD:R_0805" V 8280 2950 50  0001 C CNN
+F 2 "footprints:R_0805" V 8280 2950 50  0001 C CNN
 F 3 "" H 8350 2950 50  0001 C CNN
 	1    8350 2950
@@
 F 0 "R8" V 8250 3150 50  0000 C CNN
 F 1 "R" V 8350 3150 50  0000 C CNN
-F 2 "Resistors_SMD:R_0805" V 8280 3150 50  0001 C CNN
+F 2 "footprints:R_0805" V 8280 3150 50  0001 C CNN
 F 3 "" H 8350 3150 50  0001 C CNN
 	1    8350 3150
@@
 F 0 "BZ1" H 10850 5300 50  0000 L CNN
 F 1 "Buzzer" H 10850 5200 50  0000 L CNN
-F 2 "Buzzers_Beepers:BUZZER" V 10675 5350 50  0001 C CNN
+F 2 "footprints:BUZZER" V 10675 5350 50  0001 C CNN
 F 3 "" V 10675 5350 50  0001 C CNN
 	1    10700 5250
@@
 $EndComp
 $Comp
-L 2N4401 T1
+L 2N4401-RESCUE-microbit-extension T1
 U 1 1 59873D13
 P 10500 5650
 F 0 "T1" H 10099 5950 50  0000 L BNN
 F 1 "2N4401" H 10100 5850 50  0000 L BNN
-F 2 "TO_SOT_Packages_SMD:SOT-23" H 10500 5650 50  0001 L BNN
+F 2 "footprints:SOT-23" H 10500 5650 50  0001 L BNN
 F 3 "Multicomp" H 10500 5650 50  0001 L BNN
 F 4 "BIPOLAR TRANSISTOR%2C NPN%2C TO-92%3B Transistor Polarity%3A NPN%3B Collector Emitter Voltage V%28br%29ceo%3A 40V%3B Transition Frequen..." H 10500 5650 50  0001 L BNN "Description"
@@
 F 0 "R9" V 10280 5650 50  0000 C CNN
 F 1 "1K" V 10200 5650 50  0000 C CNN
-F 2 "Resistors_SMD:R_0805" V 10130 5650 50  0001 C CNN
+F 2 "footprints:R_0805" V 10130 5650 50  0001 C CNN
 F 3 "" H 10200 5650 50  0001 C CNN
 	1    10200 5650
@@
 F 0 "U1" H 8700 4400 50  0000 C CNN
 F 1 "LD1117S33CTR" H 8700 4350 50  0000 C CNN
-F 2 "TO_SOT_Packages_SMD:SOT-223" H 8700 4250 50  0001 C CNN
+F 2 "footprints:SOT-223" H 8700 4250 50  0001 C CNN
 F 3 "" H 8700 4150 50  0001 C CNN
 	1    8700 4150
@@
 F 0 "C1" H 8175 4500 50  0000 L CNN
 F 1 "100nF" H 8175 4300 50  0000 L CNN
-F 2 "Capacitors_SMD:C_0805" H 8188 4250 50  0001 C CNN
+F 2 "footprints:C_0805" H 8188 4250 50  0001 C CNN
 F 3 "" H 8150 4400 50  0001 C CNN
 	1    8150 4400
@@
 F 0 "C2" H 9225 4500 50  0000 L CNN
 F 1 "10uF" H 9225 4300 50  0000 L CNN
-F 2 "Capacitors_SMD:C_0805" H 9238 4250 50  0001 C CNN
+F 2 "footprints:C_0805" H 9238 4250 50  0001 C CNN
 F 3 "" H 9200 4400 50  0001 C CNN
 	1    9200 4400
@@
 F 0 "J2" H 8650 5450 50  0000 C CNN
 F 1 "9V conn" V 8750 5300 50  0000 C CNN
-F 2 "Pin_Headers:Pin_Header_Straight_1x02_Pitch2.54mm" H 8650 5300 50  0001 C CNN
+F 2 "footprints:Pin_Header_Straight_1x02_Pitch2.54mm" H 8650 5300 50  0001 C CNN
 F 3 "" H 8650 5300 50  0001 C CNN
 	1    8650 5300
